Commit message: completed code

File: src/my_robot/urdf/my_robot.xacro (robot description, xacro)
@@ -33,4 +33,9 @@
     <axis xyz="0 1 0" rpy="0 0 0" />
   </joint>
+  <joint name="camera_optical_joint" type="fixed">
+    <origin xyz="0 0 0" rpy="-1.5707 0 -1.5707"/>
+    <parent link="camera"/>
+    <child link="camera_link_optical"/>
+  </joint>
   <joint type="fixed" name="camera_joint">
     <origin xyz="0.3 0 0" rpy="0 0 0" />
@@ -146,4 +151,6 @@
     </collision>
   </link>
+  <link name="camera_link_optical">
+  </link>
   <link name="camera">
     <inertial>

Commit message: rviz config added to the rviz launch

File: src/my_robot/urdf/my_robot.xacro (robot description, xacro)
@@ -35,5 +35,6 @@
   </joint>
   <joint name="camera_optical_joint" type="fixed">
-    <origin xyz="0 0 0" rpy="-1.5707 0 -1.5707"/>
+    <!-- <origin xyz="0 0 0" rpy="-1.5707 0 -1.5707"/> -->
+    <origin xyz="0 0 0" rpy="0 0 0"/>
     <parent link="camera"/>
     <child link="camera_link_optical"/>
